Commit message: update de codigo xacro

File: src/trixy/urdf/trixy.xacro (robot description, xacro)
@@ -21,11 +21,18 @@
   </joint>
   <joint name="camera_joint" type="fixed">
-    <origin xyz="0.26 0 0" rpy="0 0 0" />
+    <origin xyz="0.17 0 0.05" rpy="0 0 0" />
     <parent link="chassis"/>
     <child link="camera" />
     <axis xyz="0 1 0"/>
   </joint>
+<!-- me he quedado cambiando la camara trasera-->
+  <joint name="camara_trasera_joint" type="fixed">
+    <origin xyz="-0.17 0 0.05" rpy="0 0 3.14" />
+    <parent link="chassis"/>
+    <child link="camara_trasera" />
+    <axis xyz="0 1 0"/>
+  </joint>
   <joint name="hokuyo_joint" type="fixed">
-    <origin xyz="0.2 0 0.2" rpy="0 0 0" />
+    <origin xyz="0.10 -0.03 0.15" rpy="0 0 0" />
     <parent link="chassis"/>
     <child link="hokuyo" />
@@ -33,5 +40,5 @@
   </joint>
   <joint type="continuous" name="left_wheel_hinge">
-    <origin xyz="0 0.30 0" rpy="0 0 0" />
+    <origin xyz="0 0.17 0" rpy="0 0 0" />
     <parent link="chassis"/>
     <child link="left_wheel" />
@@ -41,5 +48,5 @@
   </joint>
   <joint type="continuous" name="right_wheel_hinge">
-    <origin xyz="0 -0.30 0" rpy="0 0 0" />
+    <origin xyz="0 -0.17 0" rpy="0 0 0" />
     <parent link="chassis"/>
     <child link="right_wheel" />
@@ -71,7 +78,7 @@
     </visual>
   </link>
-  <link name="hokuyo">
-    <inertial>
-      <mass value="1e-5"/>
+  <link name="camara_trasera">
+    <inertial>
+      <mass value="0.1"/>
       <origin xyz="0 0 0" rpy="0 0 0"/>
       <inertia
@@ -84,4 +91,27 @@
       <origin xyz="0 0 0" rpy="0 0 0"/>
       <geometry>
+        <box size="0.05 0.05 0.05"/>
+      </geometry>
+    </collision>
+    <visual>
+      <origin xyz="0 0 0" rpy="0 0 0"/>
+      <geometry>
+        <box size="0.05 0.05 0.05"/>
+      </geometry>
+    </visual>
+  </link>
+  <link name="hokuyo">
+    <inertial>
+      <mass value="1e-5"/>
+      <origin xyz="0 0 0" rpy="0 0 0"/>
+      <inertia
+        ixx="1e-6" ixy="0.0" ixz="0.0"
+        iyy="1e-6" iyz="0.0"
+        izz="1e-6"
+      />
+    </inertial>
+    <collision>
+      <origin xyz="0 0 0" rpy="0 0 0"/>
+      <geometry>
         <box size="0.1 0.1 0.1"/>
       </geometry>
@@ -107,11 +137,11 @@
       <origin xyz="0 0 0" rpy="0 1.5707 1.5707"/>
       <geometry>
-        <cylinder radius="0.1" length="0.05"/>
-      </geometry>
-    </collision>
-    <visual>
-      <origin xyz="0 0 0" rpy="0 1.5707 1.5707"/>
-      <geometry>
-        <cylinder radius="0.1" length="0.05"/>
+        <cylinder radius="0.08" length="0.04"/>
+      </geometry>
+    </collision>
+    <visual>
+      <origin xyz="0 0 0" rpy="0 1.5707 1.5707"/>
+      <geometry>
+        <cylinder radius="0.08" length="0.04"/>
       </geometry>
     </visual>
@@ -130,11 +160,11 @@
       <origin xyz="0 0 0" rpy="0 1.5707 1.5707"/>
       <geometry>
-        <cylinder radius="0.1" length="0.05"/>
-      </geometry>
-    </collision>
-    <visual>
-      <origin xyz="0 0 0" rpy="0 1.5707 1.5707"/>
-      <geometry>
-        <cylinder radius="0.1" length="0.05"/>
+        <cylinder radius="0.08" length="0.04"/>
+      </geometry>
+    </collision>
+    <visual>
+      <origin xyz="0 0 0" rpy="0 1.5707 1.5707"/>
+      <geometry>
+        <cylinder radius="0.08" length="0.04"/>
       </geometry>
     </visual>
@@ -143,5 +173,5 @@
     <pose>0 0 0.1 0 0 0</pose>
     <inertial>
-      <mass value="15.0"/>
+      <mass value="25.0"/>
       <origin xyz="0.0 0 0" rpy=" 0 0 0"/>
       <inertia
@@ -151,8 +181,8 @@
       />
     </inertial>
-    <collision name='collision'>
+    <collision name='chassis_collision'>
       <origin xyz="0 0 0.05" rpy=" 0 0 0"/>
       <geometry>
-        <cylinder length="0.2" radius="0.25"/>
+        <box size="0.3 0.3 0.1"/>
       </geometry>
     </collision>
@@ -160,9 +190,9 @@
       <origin xyz="0 0 0.05" rpy=" 0 0 0"/>
       <geometry>
-       <cylinder length="0.2" radius="0.25"/>
+        <box size="0.3 0.3 0.1"/>
       </geometry>
     </visual>
     <collision name='back_caster_collision'>
-      <origin xyz="-0.15 0 -0.05" rpy=" 0 0 0"/>
+      <origin xyz="-0.11 0 -0.03" rpy=" 0 0 0"/>
       <geometry>
         <sphere radius="0.0499"/>
@@ -170,5 +200,5 @@
     </collision>
     <visual name='back_caster_visual'>
-      <origin xyz="-0.15 0 -0.05" rpy=" 0 0 0"/>
+      <origin xyz="-0.11 0 -0.03" rpy=" 0 0 0"/>
       <geometry>
         <sphere radius="0.05"/>
@@ -176,5 +206,5 @@
     </visual>
     <collision name='front_caster_collision'>
-      <origin xyz="0.15 0 -0.05" rpy=" 0 0 0"/>
+      <origin xyz="0.11 0 -0.03" rpy=" 0 0 0"/>
       <geometry>
         <sphere radius="0.0499"/>
@@ -182,5 +212,5 @@
     </collision>
     <visual name='front_caster_visual'>
-      <origin xyz="0.15 0 -0.05" rpy=" 0 0 0"/>
+      <origin xyz="0.11 0 -0.03" rpy=" 0 0 0"/>
       <geometry>
         <sphere radius="0.05"/>
